Commit message: autnomous driving stack up. weak point: the nav2 planner

File: src/gazebo_stuff/urdf/rover_with_lidar.urdf.xacro (robot description, xacro)
@@ -23,5 +23,5 @@
         <parent link="base_link"/>
         <child link="laser_frame"/>
-        <origin xyz="0.05 0.0 0.18" rpy="0 0 0"/>
+        <origin xyz="0.12 0.0 0.23" rpy="0 0.1745 0"/>
       </joint>
       <!-- Gazebo GPU LiDAR Sensor Plugin -->
@@ -36,15 +36,15 @@
             <scan>
               <horizontal>
-                <samples>360</samples>
+                <samples>720</samples>
                 <resolution>1</resolution>
                 <min_angle>-3.14159</min_angle>
                 <max_angle>3.14159</max_angle>
               </horizontal>
-              <!-- 16 Vertical Beams, tilted DOWN: -20 deg to +3 deg (was +/-15). Sensor ~0.38m up; dense ground 1-8m, near-horizontal beams still climb ramps/obstacles, few sky/inf rays. -->
+              <!-- 16 Vertical Beams (-15 deg to +10 deg). Sweeps terrain features & crater rims out to 15m -->
               <vertical>
                 <samples>16</samples>
                 <resolution>1</resolution>
-                <min_angle>-0.349066</min_angle>
-                <max_angle>0.052360</max_angle>
+                <min_angle>-0.2618</min_angle>
+                <max_angle>0.1745</max_angle>
               </vertical>
             </scan>
